Commit message: Fixed issue with TF and updated launch file to accept robot feedback as input

File: imr_arm_description/urdf/imr_arm_rviz.urdf (robot description, URDF)
Before this commit: robot imr_arm, 6 links, 5 joints
Links:
- removed link base_link
- added link world
Joints:
- removed joint X5-9_to_base
- removed joint base_to_link1
- removed joint link1_to_link2
- removed joint link2_to_wrist
- removed joint world_to_X5-9
- added joint Joint0: type fixed, parent world, child X5-9
- added joint Joint1: type continuous, parent X5-9, child base, origin xyz=0 0 0.031 rpy=0 0 0, axis 0 0 1
- added joint Joint2: type continuous, parent base, child link1, origin xyz=0 -0.006 0.055 rpy=0 0 0, axis 0 -1 0
- added joint Joint3: type continuous, parent link1, child link2, origin xyz=0 0.031 0.280 rpy=0 0 0, axis 0 1 0
- added joint Joint4: type continuous, parent link2, child wrist, origin xyz=0 -0.031 0.280 rpy=0 0 0, axis 0 -1 0

Commit message: Updated the gazebo and rviz environments to accept all 5 DOFs with position control on the gazebo interface

File: imr_arm_description/urdf/imr_arm_rviz.urdf (robot description, URDF)
Before this commit: robot imr_arm, 6 links, 5 joints
Links:
- added link EE, mass 0.001
Joints:
- added joint Joint5: type continuous, parent wrist, child EE, origin xyz=0 -0.04 0.07 rpy=0 0 0, axis 0 0 1
