Commit message: Added IMR tabletop, tray to manipulate, and end effectors to the arms all with appropriate contacts

File: imr_arm_description/urdf/imr_arm_gazebo.urdf (robot description, URDF)
Before this commit: robot imr_arm, 7 links, 6 joints
Links:
- link EE: geometry collision mesh filename=package://imr_arm_description/meshes/EndEffector_Contact.dae; visual mesh filename=package://imr_arm_description/meshes/EndEffector.dae
Joints:
- joint Joint5: origin xyz=0 -0.04 0.07 rpy=0 0 0 -> xyz=0 -0.04 0.0745 rpy=0 0 0

File: imr_arm_description/urdf/imr_arm_gazebo2.urdf (robot description, URDF)
Before this commit: robot imr_arm, 7 links, 6 joints
Links:
- link EE: mass 0.4014 -> 0.6416; geometry collision mesh filename=package://imr_arm_description/meshes/EndEffector_Contact.dae; visual mesh filename=package://imr_arm_description/meshes/EndEffector.dae
Joints:
- joint Joint5: limit lower=-3. upper=3. effort=2.5 velocity=9.6 -> lower=-3. upper=3. effort=7 velocity=9.6; origin xyz=0 -0.04 0.07 rpy=0 0 0 -> xyz=0 -0.04 0.0745 rpy=0 0 0
